Commit message: removed collision error

File: packages/suturo_urdf_publisher/urdf/hsr_movable_door.urdf.xacro (robot description, xacro)
@@ -18,5 +18,5 @@
       </visual>
       <collision>
-        <origin xyz="${width/2}$ ${depth/2} 0" rpy="0 0 0" />
+        <origin xyz="${width/2} ${depth/2} 0" rpy="0 0 0" />
         <geometry>
           <box size="${width} ${depth} ${height}" />
